Commit message: Added macro to create bottles pack with loops

File: hrc_case_study_descriptions/urdf/bottle.urdf.xacro (robot description, xacro)
@@ -2,12 +2,12 @@
 <!--URDF MODEL only arms-->
 <robot xmlns:xacro="http://wiki.ros.org/xacro" name="bottle">
-  <xacro:macro name="bottle" params="parent_link_name xyz rpy item">
+  <xacro:macro name="bottle" params="parent_link_name pack_name xyz rpy item">
   <joint name="base_bottle_${item}" type="fixed">
     <parent link="${parent_link_name}"/>
-    <child link="bottle_${item}_link"/>
+    <child link="bottle_${pack_name}_${item}_link"/>
     <origin xyz="${xyz}" rpy="${rpy}" />
   </joint>
     <link
-      name="bottle_${item}_link">
+      name="bottle_${pack_name}_${item}_link">
       <inertial>
         <origin

File: hrc_case_study_descriptions/urdf/sharework_cell.urdf.xacro (robot description, xacro)
@@ -422,4 +422,5 @@
   </collision>
 </link>
+<!-- Include and call the working table with wheels macro -->
 <xacro:include filename="$(find hrc_case_study_descriptions)/urdf/working_table.urdf.xacro" />
 <xacro:working_table_with_wheels
@@ -427,35 +428,10 @@
   xyz = "1.5 -1.5 0"
   rpy="0 0 -1.57079632679"/>
-<xacro:include filename="$(find hrc_case_study_descriptions)/urdf/bottle.urdf.xacro" />+
-<xacro:bottle
-  parent_link_name="working_table_top_link"
-  xyz = "0.2 0.4 0"
-  rpy="0 0 0"
-  item="1"/>
-<xacro:bottle
-  parent_link_name="working_table_top_link"
-  xyz = "0.2 0.5 0"
-  rpy="0 0 0"
-  item="2"/>
-<xacro:bottle
-  parent_link_name="working_table_top_link"
-  xyz = "0.2 0.6 0"
-  rpy="0 0 0"
-  item="3"/>
-<xacro:bottle
-  parent_link_name="working_table_top_link"
-  xyz = "0.3 0.4 0"
-  rpy="0 0 0"
-  item="4"/>
-<xacro:bottle
-  parent_link_name="working_table_top_link"
-  xyz = "0.3 0.5 0"
-  rpy="0 0 0"
-  item="5"/>
-<xacro:bottle
-  parent_link_name="working_table_top_link"
-  xyz = "0.3 0.6 0"
-  rpy="0 0 0"
-  item="6"/>
+<!-- Include bottle pack xacro macro -->
+<xacro:include filename="$(find hrc_case_study_descriptions)/urdf/bottles_pack.urdf.xacro" />
+<!-- Property with the name of yaml file with bottles locations  -->
+<xacro:property name="user_pack_yaml_file_name"    value="$(find hrc_case_study_descriptions)/config/bottle_distributions.yaml"/>
+<!-- Call the pack macro in order to create the bottles pack with the config specified in the yaml -->
+<xacro:pack parent_link_name="working_table_top_link" pack_name="user_pack" yaml_file_name="${user_pack_yaml_file_name}"/>
 </xacro:macro>
 </robot>

Commit message: Added boxes

File: hrc_case_study_descriptions/urdf/bottle.urdf.xacro (robot description, xacro)
@@ -3,5 +3,5 @@
 <robot xmlns:xacro="http://wiki.ros.org/xacro" name="bottle">
   <xacro:macro name="bottle" params="parent_link_name pack_name xyz rpy item">
-  <joint name="base_bottle_${item}" type="fixed">
+  <joint name="bottle_${pack_name}_${item}" type="fixed">
     <parent link="${parent_link_name}"/>
     <child link="bottle_${pack_name}_${item}_link"/>

File: hrc_case_study_descriptions/urdf/sharework_cell.urdf.xacro (robot description, xacro)
@@ -431,7 +431,19 @@
 <xacro:include filename="$(find hrc_case_study_descriptions)/urdf/bottles_pack.urdf.xacro" />
 <!-- Property with the name of yaml file with bottles locations  -->
-<xacro:property name="user_pack_yaml_file_name"    value="$(find hrc_case_study_descriptions)/config/bottle_distributions.yaml"/>
+<xacro:property name="user_pack_yaml_file_name"    value="$(find hrc_case_study_descriptions)/config/user_bottle_distributions.yaml"/>
+<xacro:property name="robot_pack_yaml_file_name"    value="$(find hrc_case_study_descriptions)/config/robot_bottle_distributions.yaml"/>
 <!-- Call the pack macro in order to create the bottles pack with the config specified in the yaml -->
 <xacro:pack parent_link_name="working_table_top_link" pack_name="user_pack" yaml_file_name="${user_pack_yaml_file_name}"/>
+<xacro:pack parent_link_name="robot_box_link" pack_name="robot_pack" yaml_file_name="${robot_pack_yaml_file_name}"/>
+<!-- Include and call the box macro in order to create the box -->
+<xacro:include filename="$(find hrc_case_study_descriptions)/urdf/box.urdf.xacro" />
+<xacro:box parent_link_name="rail"
+           box_name="robot_box"
+           xyz = "0 0 0"
+           rpy="0 0 0" />
+<xacro:box parent_link_name="rail"
+          box_name="human_box"
+          xyz = "0.15 2.5 0"
+          rpy="0 0 1.57079632679" />
 </xacro:macro>
 </robot>

Commit message: Added bottle color

File: hrc_case_study_descriptions/urdf/bottle.urdf.xacro (robot description, xacro)
@@ -2,5 +2,5 @@
 <!--URDF MODEL only arms-->
 <robot xmlns:xacro="http://wiki.ros.org/xacro" name="bottle">
-  <xacro:macro name="bottle" params="parent_link_name pack_name xyz rpy item">
+  <xacro:macro name="bottle" params="parent_link_name pack_name xyz rpy item color">
   <joint name="bottle_${pack_name}_${item}" type="fixed">
     <parent link="${parent_link_name}"/>
@@ -35,5 +35,5 @@
           name="">
           <color
-            rgba="0.79216 0.81961 0.93333 1" />
+            rgba="${color}" />
         </material>
       </visual>

File: hrc_case_study_descriptions/urdf/bottles_pack.urdf.xacro (robot description, xacro)
@@ -2,9 +2,9 @@
 <robot xmlns:xacro="http://wiki.ros.org/xacro" name="pack">
   <xacro:include filename="$(find hrc_case_study_descriptions)/urdf/bottle.urdf.xacro" />
-  <xacro:macro name="pack" params="parent_link_name pack_name yaml_file_name">
+  <xacro:macro name="pack" params="parent_link_name pack_name yaml_file_name color">
     <xacro:property name="yaml" value="${xacro.load_yaml(yaml_file_name)}"/>
     <xacro:property name="bottles_locations"             value="${yaml['bottles_locations']}" />
     <xacro:property name="n_bottles"             value="${yaml['n_bottles']}" />
-      <xacro:macro name="loop" params="item parent_link_name pack_name bottles_locations">
+      <xacro:macro name="loop" params="item parent_link_name pack_name bottles_locations color">
         <xacro:property name="location" value="${bottles_locations[item]}" />
         <xacro:if value="${item+1}">
@@ -14,7 +14,8 @@
             xyz = "${location['xyz']}"
             rpy="${location['rpy']}"
-            item="${item}"/>
+            item="${item}"
+            color="${color}"/>
           <!-- recursively call myself -->
-          <xacro:loop item="${item-1}" parent_link_name="${parent_link_name}" pack_name="${pack_name}" bottles_locations="${bottles_locations}" />
+          <xacro:loop item="${item-1}" parent_link_name="${parent_link_name}" pack_name="${pack_name}" bottles_locations="${bottles_locations}" color="${color}"/>
         </xacro:if>
       </xacro:macro>
@@ -23,5 +24,6 @@
                   parent_link_name="${parent_link_name}"
                   pack_name="${pack_name}"
-                  bottles_locations="${bottles_locations}"/>
+                  bottles_locations="${bottles_locations}"
+                  color="${color}"/>
   </xacro:macro>
 </robot>

File: hrc_case_study_descriptions/urdf/sharework_cell.urdf.xacro (robot description, xacro)
@@ -435,5 +435,5 @@
 <xacro:property name="both_agents_pack_yaml_file_name"    value="$(find hrc_case_study_descriptions)/config/both_agents_bottle_distributions.yaml"/>
 <!-- Call the pack macro in order to create the bottles pack with the config specified in the yaml -->
-<xacro:pack parent_link_name="working_table_top_link" pack_name="user_pack" yaml_file_name="${user_pack_yaml_file_name}"/>
+<xacro:pack parent_link_name="working_table_top_link" pack_name="user_pack" yaml_file_name="${user_pack_yaml_file_name}" color="0.79216 0.81961 0.93333 1"/>
 <!-- Util link for robot bottles pack -->
 <joint name="robot_box_util" type="fixed">
@@ -443,5 +443,5 @@
   </joint>
 <link name="robot_box_util_link"/>
-<xacro:pack parent_link_name="robot_box_util_link" pack_name="robot_pack" yaml_file_name="${robot_pack_yaml_file_name}"/>
+<xacro:pack parent_link_name="robot_box_util_link" pack_name="robot_pack" yaml_file_name="${robot_pack_yaml_file_name}" color="0.79216 0.81961 0.93333 1"/>
 <!-- Util link for both agents bottles pack -->
 <joint name="both_agents_bottles_util" type="fixed">
@@ -451,5 +451,5 @@
   </joint>
 <link name="both_agents_bottles_link"/>
-<xacro:pack parent_link_name="both_agents_bottles_link" pack_name="both_agents_pack" yaml_file_name="${both_agents_pack_yaml_file_name}"/>
+<xacro:pack parent_link_name="both_agents_bottles_link" pack_name="both_agents_pack" yaml_file_name="${both_agents_pack_yaml_file_name}" color="0.93333333 0.89019608 0.79607843  1"/>
 <!-- Include and call the box macro in order to create the boxes -->
 <xacro:include filename="$(find hrc_case_study_descriptions)/urdf/box.urdf.xacro" />
@@ -461,5 +461,5 @@
           box_name="human_box"
           xyz = "0.15 2.7 0"
-          rpy="0 0 1.57079632679" />
+          rpy="0 0 1.57079632679"/>
 </xacro:macro>
 </robot>
