Commit message: Partial solution

File: hrc_case_study_descriptions/urdf/eurobox.urdf.xacro (robot description, xacro)
@@ -12,5 +12,5 @@
     <!-- <inertial>
       <origin
-        xyz="0.2503 0.50105 0.67682"
+        xyz="0.0 0.0 0.0"
         rpy="0 0 0" />
       <mass
@@ -30,5 +30,5 @@
       <geometry>
         <mesh
-          filename="package://hrc_case_study_descriptions/mesh/eurobox.STEP" scale="0.001 0.001 0.001" />
+          filename="package://hrc_case_study_descriptions/mesh/eurobox_2.STL" scale="1 1 1" />
       </geometry>
       <material
@@ -44,5 +44,5 @@
       <geometry>
         <mesh
-          filename="package://hrc_case_study_descriptions/mesh/eurobox.STEP" scale="0.001 0.001 0.001" />
+          filename="package://hrc_case_study_descriptions/mesh/eurobox_2.STL" scale="1 1 1" />
       </geometry>
     </collision>

File: hrc_case_study_descriptions/urdf/sharework_cell.urdf.xacro (robot description, xacro)
@@ -430,8 +430,23 @@
 <xacro:include filename="$(find hrc_case_study_descriptions)/urdf/eurobox.urdf.xacro" />
 <xacro:eurobox
-  parent_link_name="world"
-  box_name="gfd"
-  xyz = "-0.3 1.5 0"
-  rpy="0 0 0.1"/>
+  parent_link_name="table"
+  box_name="1"
+  xyz = "-0.3 1.45 0.01"
+  rpy="1.57079632679 0 0"/>
+<xacro:eurobox
+  parent_link_name="table"
+  box_name="2"
+  xyz = "-0.3 1.75 0.01"
+  rpy="1.57079632679 0 0"/>
+  <xacro:eurobox
+    parent_link_name="working_table_top_link"
+    box_name="3"
+    xyz = "0.3 0.3 -0.38"
+    rpy="1.57079632679 0 0"/>
+    <xacro:eurobox
+      parent_link_name="working_table_top_link"
+      box_name="4"
+      xyz = "0.3 0.6 -0.38"
+      rpy="1.57079632679 0 0"/>
 <!-- Include bottle pack xacro macro -->
 <xacro:include filename="$(find hrc_case_study_descriptions)/urdf/bottles_pack.urdf.xacro" />

File: hrc_case_study_descriptions/urdf/working_table.urdf.xacro (robot description, xacro)
@@ -10,5 +10,5 @@
   <link
     name="working_table_with_wheels_link">
-    <inertial>
+    <!-- <inertial>
       <origin
         xyz="0.2503 0.50105 0.67682"
@@ -23,5 +23,5 @@
         iyz="-0.0022709"
         izz="5.507" />
-    </inertial>
+    </inertial> -->
     <visual>
       <origin
