Commit message: Added both agents boxes

File: hrc_case_study_descriptions/urdf/sharework_cell.urdf.xacro (robot description, xacro)
@@ -433,16 +433,32 @@
 <xacro:property name="user_pack_yaml_file_name"    value="$(find hrc_case_study_descriptions)/config/user_bottle_distributions.yaml"/>
 <xacro:property name="robot_pack_yaml_file_name"    value="$(find hrc_case_study_descriptions)/config/robot_bottle_distributions.yaml"/>
+<xacro:property name="both_agents_pack_yaml_file_name"    value="$(find hrc_case_study_descriptions)/config/both_agents_bottle_distributions.yaml"/>
 <!-- Call the pack macro in order to create the bottles pack with the config specified in the yaml -->
 <xacro:pack parent_link_name="working_table_top_link" pack_name="user_pack" yaml_file_name="${user_pack_yaml_file_name}"/>
-<xacro:pack parent_link_name="robot_box_link" pack_name="robot_pack" yaml_file_name="${robot_pack_yaml_file_name}"/>
-<!-- Include and call the box macro in order to create the box -->
+<!-- Util link for robot bottles pack -->
+<joint name="robot_box_util" type="fixed">
+    <parent link="table"/>
+    <child link="robot_box_util_link"/>
+    <origin xyz="-0.6 0.1 0.05"/>
+  </joint>
+<link name="robot_box_util_link"/>
+<xacro:pack parent_link_name="robot_box_util_link" pack_name="robot_pack" yaml_file_name="${robot_pack_yaml_file_name}"/>
+<!-- Util link for both agents bottles pack -->
+<joint name="both_agents_bottles_util" type="fixed">
+    <parent link="rail"/>
+    <child link="both_agents_bottles_link"/>
+    <origin xyz="-0.15 1.4 0"/>
+  </joint>
+<link name="both_agents_bottles_link"/>
+<xacro:pack parent_link_name="both_agents_bottles_link" pack_name="both_agents_pack" yaml_file_name="${both_agents_pack_yaml_file_name}"/>
+<!-- Include and call the box macro in order to create the boxes -->
 <xacro:include filename="$(find hrc_case_study_descriptions)/urdf/box.urdf.xacro" />
 <xacro:box parent_link_name="rail"
            box_name="robot_box"
-           xyz = "0 0 0"
-           rpy="0 0 0" />
+           xyz = "0.15 0 0"
+           rpy="0 0 1.57079632679" />
 <xacro:box parent_link_name="rail"
           box_name="human_box"
-          xyz = "0.15 2.5 0"
+          xyz = "0.15 2.7 0"
           rpy="0 0 1.57079632679" />
 </xacro:macro>

Commit message: Ready for manipulation Framework

File: hrc_case_study_descriptions/urdf/sharework_cell.urdf.xacro (robot description, xacro)
@@ -431,17 +431,24 @@
 <xacro:include filename="$(find hrc_case_study_descriptions)/urdf/bottles_pack.urdf.xacro" />
 <!-- Property with the name of yaml file with bottles locations  -->
-<xacro:property name="user_pack_yaml_file_name"    value="$(find hrc_case_study_descriptions)/config/user_bottle_distributions.yaml"/>
+<!-- <xacro:property name="user_pack_yaml_file_name"    value="$(find hrc_case_study_descriptions)/config/user_bottle_distributions.yaml"/> -->
 <xacro:property name="robot_pack_yaml_file_name"    value="$(find hrc_case_study_descriptions)/config/robot_bottle_distributions.yaml"/>
 <xacro:property name="both_agents_pack_yaml_file_name"    value="$(find hrc_case_study_descriptions)/config/both_agents_bottle_distributions.yaml"/>
+<!-- Util link for user bottles pack -->
+<joint name="user_bottles_util" type="fixed">
+    <parent link="working_table_top_link"/>
+    <child link="user_bottles_link"/>
+    <origin xyz="0.2 0.4 0.0"/>
+  </joint>
+<link name="user_bottles_link"/>
 <!-- Call the pack macro in order to create the bottles pack with the config specified in the yaml -->
-<xacro:pack parent_link_name="working_table_top_link" pack_name="user_pack" yaml_file_name="${user_pack_yaml_file_name}" color="0.79216 0.81961 0.93333 1"/>
+<!-- <xacro:pack parent_link_name="user_bottles_link" pack_name="user_pack" yaml_file_name="${user_pack_yaml_file_name}" color="0.79216 0.81961 0.93333 1"/> -->
 <!-- Util link for robot bottles pack -->
-<joint name="robot_box_util" type="fixed">
+<joint name="robot_bottles_util" type="fixed">
     <parent link="table"/>
-    <child link="robot_box_util_link"/>
+    <child link="robot_bottles_link"/>
     <origin xyz="-0.6 0.1 0.05"/>
   </joint>
-<link name="robot_box_util_link"/>
-<xacro:pack parent_link_name="robot_box_util_link" pack_name="robot_pack" yaml_file_name="${robot_pack_yaml_file_name}" color="0.79216 0.81961 0.93333 1"/>
+<link name="robot_bottles_link"/>
+<!-- <xacro:pack parent_link_name="robot_bottles_link" pack_name="robot_pack" yaml_file_name="${robot_pack_yaml_file_name}" color="0.79216 0.81961 0.93333 1"/> -->
 <!-- Util link for both agents bottles pack -->
 <joint name="both_agents_bottles_util" type="fixed">
@@ -451,10 +458,10 @@
   </joint>
 <link name="both_agents_bottles_link"/>
-<xacro:pack parent_link_name="both_agents_bottles_link" pack_name="both_agents_pack" yaml_file_name="${both_agents_pack_yaml_file_name}" color="0.93333333 0.89019608 0.79607843  1"/>
+<!-- <xacro:pack parent_link_name="both_agents_bottles_link" pack_name="both_agents_pack" yaml_file_name="${both_agents_pack_yaml_file_name}" color="0.93333333 0.89019608 0.79607843  1"/> -->
 <!-- Include and call the box macro in order to create the boxes -->
 <xacro:include filename="$(find hrc_case_study_descriptions)/urdf/box.urdf.xacro" />
 <xacro:box parent_link_name="rail"
            box_name="robot_box"
-           xyz = "0.15 0 0"
+           xyz = "0.15 0.7 0"
            rpy="0 0 1.57079632679" />
 <xacro:box parent_link_name="rail"

Commit message: commit

File: hrc_case_study_descriptions/urdf/sharework_cell.urdf.xacro (robot description, xacro)
@@ -447,5 +447,5 @@
     <parent link="table"/>
     <child link="robot_bottles_link"/>
-    <origin xyz="-0.6 0.1 0.05"/>
+    <origin xyz="-0.6 0.2 0.05"/>
   </joint>
 <link name="robot_bottles_link"/>
@@ -469,4 +469,26 @@
           xyz = "0.15 2.7 0"
           rpy="0 0 1.57079632679"/>
+<!-- box -->
+<joint name="prova_joint" type="fixed">
+    <parent link="rail"/>
+    <child link="prova"/>
+    <origin xyz="-0.2 0.8 0.0"/>
+  </joint>
+<link name="prova">
+  <inertial>
+  <mass value="1"/>
+  <inertia ixx="0.0108" ixy="0" ixz="0" iyy="0.0083" iyz="0" izz="0.0042"/>
+  </inertial>
+  <visual>
+    <geometry>
+      <box size=".1 .5 .6"/>
+    </geometry>
+  </visual>
+  <collision name="box">
+    <geometry>
+      <box size=".1 .5 .6"/>
+    </geometry>
+  </collision>
+</link>
 </xacro:macro>
 </robot>

Commit message: Ewaste Case Study first changes

File: hrc_case_study_descriptions/urdf/sharework_cell.urdf.xacro (robot description, xacro)
@@ -458,37 +458,4 @@
   </joint>
 <link name="both_agents_bottles_link"/>
-<!-- <xacro:pack parent_link_name="both_agents_bottles_link" pack_name="both_agents_pack" yaml_file_name="${both_agents_pack_yaml_file_name}" color="0.93333333 0.89019608 0.79607843  1"/> -->
-<!-- Include and call the box macro in order to create the boxes -->
-<xacro:include filename="$(find hrc_case_study_descriptions)/urdf/box.urdf.xacro" />
-<xacro:box parent_link_name="rail"
-           box_name="robot_box"
-           xyz = "0.15 0.7 0"
-           rpy="0 0 1.57079632679" />
-<xacro:box parent_link_name="rail"
-          box_name="human_box"
-          xyz = "0.15 2.7 0"
-          rpy="0 0 1.57079632679"/>
-<!-- box -->
-<joint name="prova_joint" type="fixed">
-    <parent link="rail"/>
-    <child link="prova"/>
-    <origin xyz="-0.2 0.8 0.0"/>
-  </joint>
-<link name="prova">
-  <inertial>
-  <mass value="1"/>
-  <inertia ixx="0.0108" ixy="0" ixz="0" iyy="0.0083" iyz="0" izz="0.0042"/>
-  </inertial>
-  <visual>
-    <geometry>
-      <box size=".1 .5 .6"/>
-    </geometry>
-  </visual>
-  <collision name="box">
-    <geometry>
-      <box size=".1 .5 .6"/>
-    </geometry>
-  </collision>
-</link>
 </xacro:macro>
 </robot>

Commit message: Some things

File: hrc_case_study_descriptions/urdf/sharework_cell.urdf.xacro (robot description, xacro)
@@ -426,6 +426,12 @@
 <xacro:working_table_with_wheels
   parent_link_name="world"
-  xyz = "1.5 -1.5 0"
+  xyz = "1.5 1.5 0"
   rpy="0 0 -1.57079632679"/>
+<xacro:include filename="$(find hrc_case_study_descriptions)/urdf/eurobox.urdf.xacro" />
+<xacro:eurobox
+  parent_link_name="world"
+  box_name="gfd"
+  xyz = "-0.3 1.5 0"
+  rpy="0 0 0.1"/>
 <!-- Include bottle pack xacro macro -->
 <xacro:include filename="$(find hrc_case_study_descriptions)/urdf/bottles_pack.urdf.xacro" />
@@ -458,4 +464,31 @@
   </joint>
 <link name="both_agents_bottles_link"/>
+<!-- <xacro:pack parent_link_name="both_agents_bottles_link" pack_name="both_agents_pack" yaml_file_name="${both_agents_pack_yaml_file_name}" color="0.93333333 0.89019608 0.79607843  1"/> -->
+<!-- Include and call the box macro in order to create the boxes -->
+<!-- Aggiungi un nuovo giunto tra "rail" e il nuovo link -->
+<!-- Aggiungi un nuovo link -->
+<link name="collaborative_workspace_link">
+  <visual>
+    <origin xyz="0 0 0" rpy="0 0 0" />
+    <geometry>
+      <box size="0.5 0.5 0.1" /> <!-- Dimensioni del nuovo link -->
+    </geometry>
+    <material name="LightGrey"> <!-- Materiale per il nuovo link, colore grigio chiaro -->
+      <color rgba="0.7 0.7 0.7 1"/> <!-- Colore grigio chiaro, RGBA -->
+    </material>
+  </visual>
+  <collision>
+    <origin xyz="0 0 0" rpy="0 0 0" />
+    <geometry>
+      <box size="0.5 0.5 0.1" /> <!-- Dimensioni del nuovo link per la collisione -->
+    </geometry>
+  </collision>
+</link>
+<!-- Aggiungi un nuovo giunto tra "rail" e il nuovo link -->
+<joint name="rail_to_collaborative_workspace" type="fixed">
+  <parent link="rail"/>
+  <child link="collaborative_workspace_link"/>
+  <origin xyz="0 ${rail_size_y/2} 0" rpy="0 0 0" />
+</joint>
 </xacro:macro>
 </robot>

Commit message: E waste setup ready

File: hrc_case_study_descriptions/urdf/sharework_cell.urdf.xacro (robot description, xacro)
@@ -428,67 +428,41 @@
   xyz = "1.5 1.5 0"
   rpy="0 0 -1.57079632679"/>
+<xacro:include filename="$(find hrc_case_study_descriptions)/urdf/notebook.urdf.xacro" />
+<xacro:notebook
+  parent_link_name="working_table_top_link"
+  xyz = "0.1 0.1 0.01"
+  rpy="0 0 0"/>
 <xacro:include filename="$(find hrc_case_study_descriptions)/urdf/eurobox.urdf.xacro" />
+<!-- Euroboxes in robot workspace -->
 <xacro:eurobox
   parent_link_name="table"
   box_name="1"
-  xyz = "-0.3 1.45 0.01"
+  xyz = "-0.25 1.45 0.01"
   rpy="1.57079632679 0 0"/>
 <xacro:eurobox
   parent_link_name="table"
   box_name="2"
-  xyz = "-0.3 1.75 0.01"
+  xyz = "-0.25 1.7 0.01"
   rpy="1.57079632679 0 0"/>
-  <xacro:eurobox
-    parent_link_name="working_table_top_link"
-    box_name="3"
-    xyz = "0.3 0.3 -0.38"
-    rpy="1.57079632679 0 0"/>
-    <xacro:eurobox
-      parent_link_name="working_table_top_link"
-      box_name="4"
-      xyz = "0.3 0.6 -0.38"
-      rpy="1.57079632679 0 0"/>
-<!-- Include bottle pack xacro macro -->
-<xacro:include filename="$(find hrc_case_study_descriptions)/urdf/bottles_pack.urdf.xacro" />
-<!-- Property with the name of yaml file with bottles locations  -->
-<!-- <xacro:property name="user_pack_yaml_file_name"    value="$(find hrc_case_study_descriptions)/config/user_bottle_distributions.yaml"/> -->
-<xacro:property name="robot_pack_yaml_file_name"    value="$(find hrc_case_study_descriptions)/config/robot_bottle_distributions.yaml"/>
-<xacro:property name="both_agents_pack_yaml_file_name"    value="$(find hrc_case_study_descriptions)/config/both_agents_bottle_distributions.yaml"/>
-<!-- Util link for user bottles pack -->
-<joint name="user_bottles_util" type="fixed">
-    <parent link="working_table_top_link"/>
-    <child link="user_bottles_link"/>
-    <origin xyz="0.2 0.4 0.0"/>
-  </joint>
-<link name="user_bottles_link"/>
-<!-- Call the pack macro in order to create the bottles pack with the config specified in the yaml -->
-<!-- <xacro:pack parent_link_name="user_bottles_link" pack_name="user_pack" yaml_file_name="${user_pack_yaml_file_name}" color="0.79216 0.81961 0.93333 1"/> -->
-<!-- Util link for robot bottles pack -->
-<joint name="robot_bottles_util" type="fixed">
-    <parent link="table"/>
-    <child link="robot_bottles_link"/>
-    <origin xyz="-0.6 0.2 0.05"/>
-  </joint>
-<link name="robot_bottles_link"/>
-<!-- <xacro:pack parent_link_name="robot_bottles_link" pack_name="robot_pack" yaml_file_name="${robot_pack_yaml_file_name}" color="0.79216 0.81961 0.93333 1"/> -->
-<!-- Util link for both agents bottles pack -->
-<joint name="both_agents_bottles_util" type="fixed">
-    <parent link="rail"/>
-    <child link="both_agents_bottles_link"/>
-    <origin xyz="-0.15 1.4 0"/>
-  </joint>
-<link name="both_agents_bottles_link"/>
-<!-- <xacro:pack parent_link_name="both_agents_bottles_link" pack_name="both_agents_pack" yaml_file_name="${both_agents_pack_yaml_file_name}" color="0.93333333 0.89019608 0.79607843  1"/> -->
-<!-- Include and call the box macro in order to create the boxes -->
-<!-- Aggiungi un nuovo giunto tra "rail" e il nuovo link -->
-<!-- Aggiungi un nuovo link -->
+<!-- Euroboxes in human workspace -->
+<xacro:eurobox
+  parent_link_name="working_table_top_link"
+  box_name="3"
+  xyz = "0.25 0.3 -0.38"
+  rpy="1.57079632679 0 0"/>
+<xacro:eurobox
+  parent_link_name="working_table_top_link"
+  box_name="4"
+  xyz = "0.3 0.6 -0.38"
+  rpy="1.57079632679 0 0"/>
+<!-- Collaborative worspace (central box) -->
 <link name="collaborative_workspace_link">
   <visual>
     <origin xyz="0 0 0" rpy="0 0 0" />
     <geometry>
-      <box size="0.5 0.5 0.1" /> <!-- Dimensioni del nuovo link -->
+      <box size="0.5 0.5 0.1" />
     </geometry>
-    <material name="LightGrey"> <!-- Materiale per il nuovo link, colore grigio chiaro -->
-      <color rgba="0.7 0.7 0.7 1"/> <!-- Colore grigio chiaro, RGBA -->
+    <material name="LightGrey">
+      <color rgba="0.7 0.7 0.7 1"/>
     </material>
   </visual>
@@ -496,9 +470,8 @@
     <origin xyz="0 0 0" rpy="0 0 0" />
     <geometry>
-      <box size="0.5 0.5 0.1" /> <!-- Dimensioni del nuovo link per la collisione -->
+      <box size="0.5 0.5 0.1" />
     </geometry>
   </collision>
 </link>
-<!-- Aggiungi un nuovo giunto tra "rail" e il nuovo link -->
 <joint name="rail_to_collaborative_workspace" type="fixed">
   <parent link="rail"/>

Commit message: ready for tests

File: hrc_case_study_descriptions/urdf/sharework_cell.urdf.xacro (robot description, xacro)
@@ -52,4 +52,10 @@
 <xacro:property name="beech" value="0.952941176470588	0.694117647058823	0.392156862745098 1" />
 <xacro:property name="floor" value="0.4 0.4 0.5 1" />
+<xacro:property name="advanced_table_x" value="1.00" />
+<xacro:property name="advanced_table_y" value="0.70" />
+<xacro:property name="advanced_table_z" value="0.05" />
+<xacro:property name="advanced_table2_x" value="0.2" />
+<xacro:property name="advanced_table2_y" value="1" />
+<xacro:property name="advanced_table2_z" value="0.05" />
 <link name="world"/>
 <joint name="base_to_right_leg" type="fixed">
@@ -479,4 +485,54 @@
   <origin xyz="0 ${rail_size_y/2} 0" rpy="0 0 0" />
 </joint>
+<joint name="table_to_advanced_table" type="fixed">
+  <parent link="table"/>
+  <child link="advanced_table"/>
+  <origin xyz="0 0 0" rpy="0 0 1.57"/>
+</joint>
+<joint name="adv_table_to_advanced_table2" type="fixed">
+  <parent link="advanced_table"/>
+  <child link="advanced_table_2"/>
+  <origin xyz="${advanced_table_x} ${advanced_table_y} 0" rpy="0 0 -1.57"/>
+</joint>
+<link name="advanced_table">
+   <visual>
+     <origin xyz="${0.5*advanced_table_x} ${0.5*advanced_table_y} ${0.5*advanced_table_z}" rpy="0 0 0" />
+     <geometry>
+       <box size="${advanced_table_x} ${advanced_table_y} ${advanced_table_z}" />
+     </geometry>
+     <material name="White">
+       <color rgba="1 1 1 1"/>
+     </material>
+   </visual>
+   <collision>
+     <origin xyz="${-0.5*advanced_table_x} 0 ${0.5*advanced_table_z}" rpy="0 0 0" />
+     <geometry>
+       <box size="${advanced_table_x} ${advanced_table_y} ${advanced_table_z}" />
+     </geometry>
+     <material name="White">
+       <color rgba="1 1 1 1"/>
+     </material>
+   </collision>
+</link>
+<link name="advanced_table_2">
+   <visual>
+     <origin xyz="${0.5*advanced_table2_x} ${0.5*advanced_table2_y} ${0.5*advanced_table2_z}" rpy="0 0 0" />
+     <geometry>
+       <box size="${advanced_table2_x} ${advanced_table2_y} ${advanced_table2_z}" />
+     </geometry>
+     <material name="White">
+       <color rgba="1 1 1 1"/>
+     </material>
+   </visual>
+   <collision>
+     <origin xyz="${advanced_table2_x} ${advanced_table2_y} ${advanced_table2_z}" rpy="0 0 0" />
+     <geometry>
+       <box size="${advanced_table2_x} ${advanced_table2_y} ${advanced_table2_z}" />
+     </geometry>
+     <material name="White">
+       <color rgba="1 1 1 1"/>
+     </material>
+   </collision>
+</link>
 </xacro:macro>
 </robot>

Commit message: Added mao to urdf

File: hrc_case_study_descriptions/urdf/sharework_cell.urdf.xacro (robot description, xacro)
@@ -535,4 +535,11 @@
    </collision>
 </link>
+<xacro:include filename="$(find hrc_simulator_descriptions)/urdf/human14dof/human14dof.urdf.xacro"/>
+<xacro:human14dof/>
+<joint name="human_fixed_joint" type="fixed">
+  <parent link="world" />
+  <child  link = "origin_human14dof" />
+  <origin xyz="1.5 -0.2 0.0" rpy="0 0 ${pi}" />
+</joint>
 </xacro:macro>
 </robot>

Commit message: Some little changes joints, tp params mongo cell

File: hrc_case_study_descriptions/urdf/sharework_cell.urdf.xacro (robot description, xacro)
@@ -53,9 +53,9 @@
 <xacro:property name="floor" value="0.4 0.4 0.5 1" />
 <xacro:property name="advanced_table_x" value="1.00" />
-<xacro:property name="advanced_table_y" value="0.70" />
-<xacro:property name="advanced_table_z" value="0.05" />
-<xacro:property name="advanced_table2_x" value="0.2" />
+<xacro:property name="advanced_table_y" value="0.80" />
+<xacro:property name="advanced_table_z" value="0.15" />
+<xacro:property name="advanced_table2_x" value="0.3" />
 <xacro:property name="advanced_table2_y" value="1" />
-<xacro:property name="advanced_table2_z" value="0.05" />
+<xacro:property name="advanced_table2_z" value="0.15" />
 <link name="world"/>
 <joint name="base_to_right_leg" type="fixed">

Commit message: Simulations ok

File: hrc_case_study_descriptions/urdf/sharework_cell.urdf.xacro (robot description, xacro)
@@ -506,5 +506,5 @@
    </visual>
    <collision>
-     <origin xyz="${-0.5*advanced_table_x} 0 ${0.5*advanced_table_z}" rpy="0 0 0" />
+     <origin xyz="${0.5*advanced_table_x} ${0.5*advanced_table_y} ${0.5*advanced_table_z}" rpy="0 0 0" />
      <geometry>
        <box size="${advanced_table_x} ${advanced_table_y} ${advanced_table_z}" />
@@ -526,5 +526,5 @@
    </visual>
    <collision>
-     <origin xyz="${advanced_table2_x} ${advanced_table2_y} ${advanced_table2_z}" rpy="0 0 0" />
+     <origin xyz="${0.5*advanced_table2_x} ${0.5*advanced_table2_y} ${0.5*advanced_table2_z}" rpy="0 0 0" />
      <geometry>
        <box size="${advanced_table2_x} ${advanced_table2_y} ${advanced_table2_z}" />
